File: board/bb(v1).sch (EAGLE design)
At the start: 1 part

Commit message: Adição do módulo bluetooth na placa
Parts:
- removed R1: (no value), rcl:R-EU_R0805W
- added C1, C11, C12, C2: 12pF, Nordic_nRF:CAPACITOR_0402_N
- added C10: 1.0µF, Nordic_nRF:CAPACITOR_0603_N
- added C3: 0.8pF, Nordic_nRF:CAPACITOR_0402_N
- added C4, C5, C8: 100nF, Nordic_nRF:CAPACITOR_0402_N
- added C6: N.M., Nordic_nRF:CAPACITOR_0402_N
- added C7: 100pF, Nordic_nRF:CAPACITOR_0402_N
- added C9: 4.7µF, Nordic_nRF:CAPACITOR_0603_N
- added L1: 3.9nH, Nordic_nRF:INDUCTOR_0402_N
- added U1: NRF52832, Nordic_nRF:NRF52832
- added X1: 32MHz, Nordic_nRF:XTAL_32MHZ
- added X2: 32.768kHz, Nordic_nRF:XTAL_32KHZ
Connections:
- new net ANT: C3.1, L1.1, U1.ANT@30
- new net DEC1: C4.1, U1.DEC1@01
- new net DEC2: C6.1, U1.DEC2@32
- new net DEC3: C7.1, U1.DEC3@33
- new net DEC4: C10.1, U1.DEC4@46
- new net GND: C1.2, C10.2, C11.1, C12.1, C2.2, C3.2, C4.2, C5.2, C6.2, C7.2, C8.2, C9.2, U1.VSS@31, U1.VSS@45, X1.2, X1.4
- new net N$3: C2.1, U1.XC2@35, X1.3
- new net P0.00/XL1: C11.2, U1.P0.00/XL1@02, X2.1
- new net P0.01/XL2: C12.2, U1.P0.01/XL2@03, X2.2
- new net P0.02: U1.P0.02/AIN0@04
- new net P0.03: U1.P0.03/AIN1@05
- new net P0.04: U1.P0.04/AIN2@06
- new net P0.05: U1.P0.05/AIN3@07
- new net P0.06: U1.P0.06@08
- new net P0.07: U1.P0.07@09
- new net P0.08: U1.P0.08@10
- new net P0.09: U1.P0.09/NFC1@11
- new net P0.10: U1.P0.10/NFC2@12
- new net P0.11: U1.P0.11@14
- new net P0.12: U1.P0.12@15
- new net P0.13: U1.P0.13@16
- new net P0.14: U1.P0.14@17
- new net P0.15: U1.P0.15@18
- new net P0.16: U1.P0.16@19
- new net P0.17: U1.P0.17@20
- new net P0.18/SWO: U1.P0.18/SWO@21
- new net P0.19: U1.P0.19@22
- new net P0.20: U1.P0.20@23
- new net P0.21/RESET: U1.P0.21/RESET@24
- new net P0.22: U1.P0.22@27
- new net P0.23: U1.P0.23@28
- new net P0.24: U1.P0.24@29
- new net P0.25: U1.P0.25@37
- new net P0.26: U1.P0.26@38
- new net P0.27: U1.P0.27@39
- new net P0.28: U1.P0.28@40
- new net P0.29: U1.P0.29@41
- new net P0.30: U1.P0.30@42
- new net P0.31: U1.P0.31@43
- new net RF: L1.2
- new net SWDCLK: U1.SWDCLK@25
- new net SWDIO: U1.SWDIO@26
- new net VDD_P3V3: C5.1, C8.1, C9.1, U1.VDD@13, U1.VDD@36, U1.VDD@48
- new net X1: C1.1, U1.XC1@34, X1.1
